File: project/project.kicad_sch (KiCad schematic)
At the start: 22 parts, among them J1 292304-1, SW1 SW_SPDT, SW2 SW_Push_Dual, U1 SN74HC109N, U2 74HC14, U3 74HC00, U4 SN74LS139AN

Commit message: kicad
Parts:
- added U10, U11, U12, U5, U6, U7, U8, U9: SN74HC109N, DIP794W45P254L1969H508Q16, symbol JK FLIP-FLOP SN74HC109N:SN74HC109N
- added U13: AT27C512R-45PU, AT27C512R-45PU:DIP254P1524X482-28, symbol AT27C512R-45PU:AT27C512R-45PU
- added U14, U15, U16, U17, U18, U19, U20, U21, U22: 74HC273, symbol 74xx:74HC273
- added U23, U24: 74HC14, symbol 74xx:74HC14
Connections:
- net at C1_C1.2, C1_C2.2, C1_C3.2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: now also U10.8 (GND), U11.8 (GND), U12.8 (GND), U13.14 (GND), U14.10 (GND), U15.10 (GND), U16.10 (GND), U17.10 (GND), U18.10 (GND), U19.10 (GND), U20.10 (GND), U21.10 (GND), U22.10 (GND), U23.7 (GND), U24.7 (GND), U5.8 (GND), U6.8 (GND), U7.8 (GND), U8.8 (GND), U9.16 (VCC)
- net at C1_N1.7 (DISCH), C1_Ra1.2, RV1.2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: now also U10.1 (1~CLR), U10.11 (2~PRE), U10.14 (2J), U10.15 (2~CLR), U10.16 (VCC), U10.2 (1J), U10.5 (1~PRE), U11.1 (1~CLR), U11.11 (2~PRE), U11.14 (2J), U11.15 (2~CLR), U11.16 (VCC), U11.2 (1J), U11.5 (1~PRE), U12.1 (1~CLR), U12.11 (2~PRE), U12.14 (2J), U12.15 (2~CLR), U12.16 (VCC), U12.2 (1J), U12.5 (1~PRE), U13.28 (VCC), U14.20 (VCC), U15.20 (VCC), U16.20 (VCC), U17.20 (VCC), U18.20 (VCC), U19.20 (VCC), U20.20 (VCC), U21.20 (VCC), U22.1 (~{Mr}), U22.20 (VCC), U23.14 (VCC), U24.14 (VCC), U5.1 (1~CLR), U5.11 (2~PRE), U5.14 (2J), U5.15 (2~CLR), U5.16 (VCC), U5.2 (1J), U5.5 (1~PRE), U6.1 (1~CLR), U6.11 (2~PRE), U6.14 (2J), U6.15 (2~CLR), U6.16 (VCC), U6.2 (1J), U6.5 (1~PRE), U7.1 (1~CLR), U7.11 (2~PRE), U7.14 (2J), U7.15 (2~CLR), U7.16 (VCC), U7.2 (1J), U7.5 (1~PRE), U8.1 (1~CLR), U8.11 (2~PRE), U8.14 (2J), U8.15 (2~CLR), U8.16 (VCC), U8.2 (1J), U8.5 (1~PRE), U9.11 (2~PRE), U9.13 (2~K), U9.14 (2J), U9.2 (1J), U9.3 (1~K), U9.5 (1~PRE), U9.8 (GND)
- net at U2.5: now also U4.4 (1Y0)
- net at U2.6: now also U5.4 (1CLK)
- net at U1.12 (2CLK): now also U1.7 (1~Q); no longer U2.8
- net at U1.6 (1Q), U4.2 (1A): no longer U2.9
- net at U2.13: now also U4.7 (1Y3)
- net at U2.3: now also U4.5 (1Y1)
- net at U2.4: now also U22.11 (Cp)
- net at U4.6 (1Y2): now also U2.11
- new net: U7.12 (2CLK), U7.7 (1~Q)
- new net: U6.9 (2~Q), U7.4 (1CLK)
- new net: U7.9 (2~Q), U8.4 (1CLK)
- new net: U12.12 (2CLK), U12.7 (1~Q)
- new net: U11.9 (2~Q), U12.4 (1CLK)
- new net: U6.12 (2CLK), U6.7 (1~Q)
- new net: U5.9 (2~Q), U6.4 (1CLK)
- new net: U5.12 (2CLK), U5.7 (1~Q)
- new net: U11.12 (2CLK), U11.7 (1~Q)
- new net: U10.9 (2~Q), U11.4 (1CLK)
- new net: U10.12 (2CLK), U10.7 (1~Q)
- new net: U8.12 (2CLK), U8.7 (1~Q)
- new net 0: U13.10 (A0), U13.11 (O0), U14.3 (D0), U15.3 (D0), U16.3 (D0), U17.3 (D0), U18.3 (D0), U19.3 (D0), U20.3 (D0), U21.3 (D0), U22.2 (Q0), U22.3 (D0), U5.6 (1Q)
- new net 1: U13.12 (O1), U13.9 (A1), U14.4 (D1), U15.4 (D1), U16.4 (D1), U17.4 (D1), U18.4 (D1), U19.4 (D1), U20.4 (D1), U21.4 (D1), U22.4 (D1), U22.5 (Q1), U5.10 (2Q)
- new net 10: U10.6 (1Q), U13.21 (A10)
- new net 11: U10.10 (2Q), U13.23 (A11)
- new net 12: U11.6 (1Q), U13.2 (A12)
- new net 13: U11.10 (2Q), U13.26 (A13)
- new net 14: U12.6 (1Q), U13.27 (A14)
- new net 15: U12.10 (2Q), U13.1 (A15)
- new net 2: U13.13 (O2), U13.8 (A2), U14.7 (D2), U15.7 (D2), U16.7 (D2), U17.7 (D2), U18.7 (D2), U19.7 (D2), U20.7 (D2), U21.7 (D2), U22.6 (Q2), U22.7 (D2), U6.6 (1Q)
- new net 3: U13.15 (O3), U13.7 (A3), U14.8 (D3), U15.8 (D3), U16.8 (D3), U17.8 (D3), U18.8 (D3), U19.8 (D3), U20.8 (D3), U21.8 (D3), U22.8 (D3), U22.9 (Q3), U6.10 (2Q)
- new net 4: U13.16 (O4), U13.6 (A4), U14.13 (D4), U15.13 (D4), U16.13 (D4), U17.13 (D4), U18.13 (D4), U19.13 (D4), U20.13 (D4), U21.13 (D4), U22.12 (Q4), U22.13 (D4), U7.6 (1Q)
- new net 5: U13.17 (O5), U13.5 (A5), U14.14 (D5), U15.14 (D5), U16.14 (D5), U17.14 (D5), U18.14 (D5), U19.14 (D5), U20.14 (D5), U21.14 (D5), U22.14 (D5), U22.15 (Q5), U7.10 (2Q)
- new net 6: U13.18 (O6), U13.4 (A6), U14.17 (D6), U15.17 (D6), U16.17 (D6), U17.17 (D6), U18.17 (D6), U19.17 (D6), U20.17 (D6), U21.17 (D6), U22.16 (Q6), U22.17 (D6), U8.6 (1Q)
- new net 7: U13.19 (O7), U13.3 (A7), U14.18 (D7), U15.18 (D7), U16.18 (D7), U17.18 (D7), U18.18 (D7), U19.18 (D7), U20.18 (D7), U21.18 (D7), U22.18 (D7), U22.19 (Q7), U8.10 (2Q)
- new net 8: U13.25 (A8)
- new net 9: U13.24 (A9)
Other:
- note added: "instruction"
- note added: "instructions_1XXXXRRR"
- note added: "pc 1-2"
- note added: "pc 11-12"
- note added: "pc 13-14"
- note added: "pc 15-16"
- note added: "pc 3-4"
- note added: "pc 5-6"
- note added: "pc 7-8"
- note added: "pc 9-10"
- moved on the sheet: U2B, U2C, U2E, U2F

Commit message: kicad
Connections:
- net 8: now also U9.6 (1Q)
- net 9: now also U9.10 (2Q)
- net at C1_C1.2, C1_C2.2, C1_C3.2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: now also U9.8 (GND); no longer U9.16 (VCC)
- net at C1_N1.7 (DISCH), C1_Ra1.2, RV1.2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: now also U9.1 (1~CLR), U9.15 (2~CLR), U9.16 (VCC); no longer U9.13 (2~K), U9.3 (1~K), U9.8 (GND)
- net at U10.4 (1CLK): now also U9.9 (2~Q)
- net at U9.12 (2CLK): now also U9.7 (1~Q)
- net at U9.4 (1CLK): now also U8.9 (2~Q)
